File: hardware/v4/Arm Board V4.sch (EAGLE design)
At the start: 51 parts, among them IC3 L6206D, U1 SN74LS241DW, U2 XBEE-1B3, U3 LSM9DS0

Commit message: Added motor controller and cleaned it up
Parts:
- C2: device SparkFun-Capacitors:0.1UF-25V(+80/-20%)(0603) -> SparkFun-Passives:CAP1206
- C4, C9: device SparkFun-Capacitors:0.1UF-25V-5%(0603) -> SparkFun-Passives:CAP1206
- R15, R8: device SparkFun-Passives:RESISTOR0805-RES -> SparkFun-Resistors:RESISTOR1206
Changed lines of the file:
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@@
 <?xml version="1.0" encoding="utf-8"?>
 <!DOCTYPE eagle SYSTEM "eagle.dtd">
-<eagle version="7.1.0">
+<eagle version="6.5.0">
 <drawing>
 <settings>
@@
 <part name="GND44" library="SparkFun-Aesthetics" deviceset="GND" device=""/>
 <part name="GND46" library="SparkFun-Aesthetics" deviceset="GND" device=""/>
-<part name="R8" library="SparkFun-Passives" deviceset="RESISTOR" device="0805-RES" value="100k"/>
-<part name="C2" library="SparkFun-Capacitors" deviceset="0.1UF-25V(+80/-20%)(0603)" device="" value="5.6nF"/>
+<part name="R8" library="SparkFun-Resistors" deviceset="RESISTOR" device="1206" value="100k"/>
+<part name="C2" library="SparkFun-Passives" deviceset="CAP" device="1206" value="5.6nF"/>
 <part name="GND47" library="SparkFun-Aesthetics" deviceset="GND" device=""/>
 <part name="D2" library="SparkFun-DiscreteSemi" deviceset="DIODE" device="1N4148" value="1N4148"/>
 <part name="D1" library="SparkFun-DiscreteSemi" deviceset="DIODE" device="1N4148" value="1N4148"/>
-<part name="C4" library="SparkFun-Capacitors" deviceset="0.1UF-25V-5%(0603)" device="" value="220nF"/>
-<part name="C9" library="SparkFun-Capacitors" deviceset="0.1UF-25V-5%(0603)" device="" value="10nF"/>
-<part name="R15" library="SparkFun-Passives" deviceset="RESISTOR" device="0805-RES" value="100"/>
+<part name="C4" library="SparkFun-Passives" deviceset="CAP" device="1206" value="220nF"/>
+<part name="C9" library="SparkFun-Passives" deviceset="CAP" device="1206" value="10nF"/>
+<part name="R15" library="SparkFun-Resistors" deviceset="RESISTOR" device="1206" value="100"/>
 </parts>
 <sheets>
